File: PCB/_autosave-TCRHMAG.kicad_sch (KiCad schematic)
At the start: 31 parts, among them J1 CONN_BATTERY, J2 CONN_LED, J3 CONN_THERM, J4 CONN_OLED, J5 CONN_HEATER, Q301 Si4116DY, SW101 PWR_SW, U101 L78L05_SOT89, U102 CH32V003FxPx

Commit message: Added OpAmp GPIO and init functions
Connections:
- net MCU_OPAMP_OUT renamed MCU_OPAMP_ADC
Changed lines of the file:
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@@
 		)
 	)
-	(label "MCU_OPAMP_OUT"
+	(label "MCU_OPAMP_ADC"
 		(at 120.65 149.225 180)
 		(effects
@@
 		)
 	)
-	(label "MCU_OPAMP_OUT"
+	(label "MCU_OPAMP_ADC"
 		(at 215.265 116.84 180)
 		(effects
@@
 		)
 	)
-	(label "MCU_OPAMP_OUT"
+	(label "MCU_OPAMP_ADC"
 		(at 281.305 116.84 180)
 		(effects
