File: PCB/TCRHMAG.kicad_pcb (KiCad board)
At the start: 2 copper layers, 42.8 x 37.1 mm, 33 parts, among them J1 CONN_BATTERY, J2 CONN_LED, J3 CONN_THERM, J4 CONN_OLED, J5 CONN_HEATER, J6 CONN_ENCODER, J7 CONN_PROG, Q301 Si4116DY, SW101 PWR_SW, U101 L78L05_SOT89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

Commit message: MkIII PCB Finished
Parts:
- added C105: 10uF, Capacitor_SMD:C_0402_1005Metric, B.Cu at (82.7, 61.1)
- added C106: 10nF, Capacitor_SMD:C_0402_1005Metric, B.Cu at (77.9, 82.7)
- added C107: 10nF, Capacitor_SMD:C_0402_1005Metric, B.Cu at (77.9, 81.7)
- added R109: 4K7, Resistor_SMD:R_0402_1005Metric, B.Cu at (77.9, 79.7)
- added R110: 4K7, Resistor_SMD:R_0402_1005Metric, B.Cu at (77.9, 80.7)
- added R111: 4K7, Resistor_SMD:R_0402_1005Metric, B.Cu at (77.9, 83.7)
- added R112: 4K7, Resistor_SMD:R_0402_1005Metric, B.Cu at (77.9, 84.7)
- C101, C102, C103, C104, C201: footprint Capacitor_SMD:C_0603_1608Metric -> Capacitor_SMD:C_0402_1005Metric
- C301, C302: footprint Capacitor_SMD:C_0603_1608Metric -> Capacitor_SMD:C_0402_1005Metric; moved to B.Cu
- J4, J6: footprint Connector_PinHeader_1.00mm:PinHeader_1x04_P1.00mm_Vertical -> Connector_PinSocket_2.00mm:PinSocket_1x04_P2.00mm_Vertical
- R101, R102, R103, R104, R201, R202, R203, R204: footprint Resistor_SMD:R_0603_1608Metric -> Resistor_SMD:R_0402_1005Metric
- R105, R106, R107, R108, R303: footprint Resistor_SMD:R_0603_1608Metric -> Resistor_SMD:R_0402_1005Metric; moved to B.Cu
- moved J4 13.6 mm to (89.5, 84.3), turned to -90 degrees
- moved J6 7.80 mm to (83.5, 80.3), turned to 90 degrees
- moved C301 5.80 mm to (91.3, 76.8)
- moved C302 5.41 mm to (89.8, 77.3), turned to 90 degrees
- moved R107 4.84 mm to (77.9, 85.7)
- moved C104 4.63 mm to (77.9, 78.7)
- moved R108 4.51 mm to (77.9, 86.7)
- moved R101 4.40 mm to (82.2, 59.5)
- moved C101 4.31 mm to (83.2, 59.5)
- moved R102 4.20 mm to (82.2, 62.7)
- moved U101 4.19 mm to (86.7, 61.1)
- moved C102 4.11 mm to (83.2, 62.7)
- moved R303 3.89 mm to (91.3, 77.8)
- moved R105 3.68 mm to (91.3, 74.8), turned to 0 degrees
- moved R201 2.22 mm to (77.9, 77.7)
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Connections:
- net /BATTERY_FILL renamed Net-(J1-Pin_2)
- net /HEATER_FILL renamed Net-(J5-Pin_2)
- J4 pad 2: /MCU_SDA -> /MCU_SCL
- J4 pad 3: /MCU_SCL -> /MCU_SDA
- J6 pad 2: /MCU_ENC_A -> Net-(J6-Pin_2)
- J6 pad 3: /MCU_ENC_B -> Net-(J6-Pin_3)
- R107 pad 2: /MCU_SDA -> /MCU_SCL
- R108 pad 2: /MCU_SCL -> /MCU_SDA
Routing:
- net Net-(J1-Pin_2): track 0.00 -> 27.8 mm
- net /PBUS_5V: track 78.2 -> 98.5 mm, vias 4 -> 5
- net /PBUS_BATT: track 5.25 -> 25.4 mm
- net /MCU_OPAMP_CH1+: track 16.1 -> 31.7 mm, vias 1 -> 0
- net /MCU_HEATER_OUT: track 20.8 -> 35.9 mm, vias 1 -> 0
- net /MCU_THERM_IN: track 37.0 -> 49.9 mm
- net Net-(J6-Pin_3): track 0.00 -> 11.3 mm
- net /CSENSE_FILL: track 0.00 -> 10.1 mm, vias 0 -> 2
- net /MCU_ENC_A: track 22.5 -> 12.9 mm
- net Net-(J6-Pin_2): track 0.00 -> 9.07 mm
- net /MCU_ENC_SW: track 17.0 -> 25.5 mm, vias 0 -> 1
- net /MCU_ENC_B: track 19.8 -> 13.1 mm
- net GND: track 25.0 -> 20.6 mm, vias 71 -> 73
- net /MCU_SCL: track 21.5 -> 25.8 mm, vias 0 -> 1
- net /MCU_SDA: track 19.8 -> 23.9 mm, vias 0 -> 1
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- removed copper zone on F.Cu, net /PBUS_BATT
- removed copper zone on F.Cu, net Net-(J1-Pin_2)
Other:
- board text added: "TCRHMAG Controller MkIII 25 May 2026"
- board text removed: "TCRHMAG Controller MkII 19 Mar 2026"

Commit message: PCB MkIII Final version gerber output. Changed gitignore
Routing:
- net GND: track 20.6 -> 21.3 mm, vias 73 -> 76
Other:
- board text added: "TCRHMAG Controller MkIII 27 May 2026"
- board text removed: "TCRHMAG Controller MkIII 25 May 2026"
Changed lines of the file:
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@@
 			(drillshape 0)
 			(scaleselection 1)
-			(outputdirectory "Gerb/")
+			(outputdirectory "/home/ash/Development/CH32V00x/TCRHMAG/PCB/Gerb")
 		)
 	)
@@
 		)
 		(fp_text user "${REFERENCE}"
-			(at 0 -6.1 0)
+			(at 0 -8.4 0)
 			(unlocked yes)
 			(layer "F.Fab")
@@
 		)
 		(fp_text user "${REFERENCE}"
-			(at 0 -6.2 0)
+			(at 0 -8.4 0)
 			(unlocked yes)
 			(layer "F.Fab")
@@
 	)
 	(gr_text "+ LED -"
-		(at 93.1 60.3 0)
+		(at 93.1 60.4 0)
 		(layer "F.SilkS")
 		(effects
@@
 	)
 	(gr_text "HEATER"
-		(at 104.4 70.3 270)
+		(at 104.5 70.3 90)
 		(layer "F.SilkS")
 		(effects
@@
 		)
 	)
-	(gr_text "TCRHMAG Controller\nMkIII   25 May 2026"
+	(gr_text "TCRHMAG Controller\nMkIII   27 May 2026"
 		(at 71.7 90.3 9.8)
 		(layer "B.SilkS")
@@
 		(start 89.5 77.8)
 		(end 89.2 77.5)
-		(width 0.4)
+		(width 0.6)
 		(layer "F.Cu")
 		(net "/CSENSE_FILL")
@@
 		(start 92.4 76.8)
 		(end 89.675 76.8)
-		(width 0.4)
+		(width 0.6)
 		(layer "F.Cu")
 		(net "/CSENSE_FILL")
@@
 		(start 89.2 76.375)
 		(end 89.225 76.35)
-		(width 0.4)
+		(width 0.6)
 		(layer "F.Cu")
 		(net "/CSENSE_FILL")
@@
 		(start 89.2 77.5)
 		(end 89.2 76.375)
-		(width 0.4)
+		(width 0.6)
 		(layer "F.Cu")
 		(net "/CSENSE_FILL")
@@
 		(start 89.675 76.8)
 		(end 89.225 76.35)
-		(width 0.4)
+		(width 0.6)
 		(layer "F.Cu")
 		(net "/CSENSE_FILL")
@@
 		(start 92.4 77.8)
 		(end 89.5 77.8)
-		(width 0.4)
+		(width 0.6)
 		(layer "F.Cu")
 		(net "/CSENSE_FILL")
@@
 		(start 91.81 77.8)
 		(end 92.4 77.8)
-		(width 0.4)
+		(width 0.6)
 		(layer "B.Cu")
 		(net "/CSENSE_FILL")
@@
 		(start 91.78 76.8)
 		(end 92.4 76.8)
-		(width 0.4)
+		(width 0.6)
 		(layer "B.Cu")
 		(net "/CSENSE_FILL")
@@
 		(start 91.78 77.77)
 		(end 91.81 77.8)
-		(width 0.4)
+		(width 0.6)
 		(layer "B.Cu")
 		(net "/CSENSE_FILL")
@@
 		(start 91.78 76.8)
 		(end 91.78 77.77)
-		(width 0.4)
+		(width 0.6)
 		(layer "B.Cu")
 		(net "/CSENSE_FILL")
@@
 	)
 	(via
+		(at 100.8 76.1)
+		(size 0.6)
+		(drill 0.3)
+		(layers "F.Cu" "B.Cu")
+		(free yes)
+		(net "GND")
+	)
+	(via
 		(at 84.4 72.845)
 		(size 0.7)
@@
 	)
 	(via
+		(at 75.2 72.8)
+		(size 0.6)
+		(drill 0.3)
+		(layers "F.Cu" "B.Cu")
+		(free yes)
+		(net "GND")
+	)
+	(via
 		(at 66.7 91.8)
 		(size 0.6)
@@
 	)
 	(via
-		(at 72.8 77.7)
+		(at 72.3 77)
 		(size 0.6)
 		(drill 0.3)
@@
 	)
 	(via
+		(at 104.3 70.1)
+		(size 0.6)
+		(drill 0.3)
+		(layers "F.Cu" "B.Cu")
+		(free yes)
+		(net "GND")
+	)
+	(via
 		(at 86.4 75.845)
 		(size 0.7)
@@
 	)
 	(segment
-		(start 73 77.5)
-		(end 72.8 77.7)
+		(start 72.8 77.5)
+		(end 74.125 77.5)
 		(width 0.4)
 		(layer "B.Cu")
@@
 	)
 	(segment
+		(start 72.3 77)
+		(end 72.8 77.5)
+		(width 0.4)
+		(layer "B.Cu")
+		(net "GND")
+	)
+	(segment
 		(start 76 77.5)
 		(end 74.125 77.5)
@@
 	)
 	(segment
-		(start 74.125 77.5)
-		(end 73 77.5)
-		(width 0.4)
-		(layer "B.Cu")
-		(net "GND")
-	)
-	(segment
 		(start 90.8 76.82)
 		(end 90.82 76.8)
@@
 	)
 	(segment
-		(start 76.87868 72.12132)
+		(start 76 74.242641)
+		(end 75.999995 73.906245)
+		(width 0.4)
+		(layer "F.Cu")
+		(net "/MCU_BATT_VSENS")
+	)
+	(segment
+		(start 76.640783 72.359217)
 		(end 80.521321 68.478679)
 		(width 0.4)
@@
 	)
 	(arc
-		(start 76 74.242641)
-		(mid 76.228362 73.09459)
-		(end 76.87868 72.12132)
+		(start 75.999995 73.906245)
+		(mid 76.166525 73.068999)
+		(end 76.640783 72.359217)
 		(width 0.4)
 		(layer "F.Cu")
